Commit message: test launch files

File: demo_packages/velodyne_simulator/urdf/HDL-32E.urdf.xacro (robot description, xacro)
@@ -18,5 +18,5 @@
       <visual>
         <geometry>
-          <mesh filename="package://tel211/velodyne_simulator_pkgs/meshes/HDL32E_base.dae" />
+          <mesh filename="package://demo_packages/velodyne_simulator/meshes/HDL32E_base.dae" />
         </geometry>
       </visual>
@@ -42,5 +42,5 @@
         <origin xyz="0 0 -0.09081" rpy="0 0 0" />
         <geometry>
-          <mesh filename="package://tel211/velodyne_simulator_pkgs/meshes/HDL32E_scan.dae" />
+          <mesh filename="package://demo_packages/velodyne_simulator/meshes/HDL32E_scan.dae" />
         </geometry>
       </visual>

File: demo_packages/velodyne_simulator/urdf/VLP-16.urdf.xacro (robot description, xacro)
@@ -18,10 +18,10 @@
       <visual>
         <geometry>
-          <mesh filename="package://tel211/velodyne_simulator_pkgs/meshes/VLP16_base_1.dae" />
+          <mesh filename="package://demo_packages/velodyne_simulator/meshes/VLP16_base_1.dae" />
         </geometry>
       </visual>
       <visual>
         <geometry>
-          <mesh filename="package://tel211/velodyne_simulator_pkgs/meshes/VLP16_base_2.dae" />
+          <mesh filename="package://demo_packages/velodyne_simulator/meshes/VLP16_base_2.dae" />
         </geometry>
       </visual>
@@ -47,5 +47,5 @@
         <origin xyz="0 0 -0.0377" />
         <geometry>
-          <mesh filename="package://tel211/velodyne_simulator_pkgs/meshes/VLP16_scan.dae" />
+          <mesh filename="package://demo_packages/velodyne_simulator/meshes/VLP16_scan.dae" />
         </geometry>
       </visual>

File: demo_packages/velodyne_simulator/urdf/example.urdf.xacro (robot description, xacro)
@@ -32,9 +32,9 @@
     </inertial>
   </link>
-  <xacro:include filename="$(find tel211)/velodyne_simulator_pkgs/urdf/VLP-16.urdf.xacro"/>
+  <xacro:include filename="$(find demo_packages)/velodyne_simulator/urdf/VLP-16.urdf.xacro"/>
   <xacro:VLP-16 parent="base_link" name="velodyne" topic="/velodyne_points" organize_cloud="${organize_cloud}" hz="10" samples="440" gpu="${gpu}">
     <origin xyz="0 0 0.4" rpy="0 0 0" />
   </xacro:VLP-16>
-  <xacro:include filename="$(find tel211)/velodyne_simulator_pkgs/urdf/HDL-32E.urdf.xacro"/>
+  <xacro:include filename="$(find demo_packages)/velodyne_simulator/urdf/HDL-32E.urdf.xacro"/>
   <xacro:HDL-32E parent="base_link" name="velodyne2" topic="/velodyne_points2" organize_cloud="${organize_cloud}" hz="10" samples="220" gpu="${gpu}">
     <origin xyz="0 0 0.6" rpy="0 0 0" />
